File: KiCad_Projects/psu_board/psu_board/psu_board.kicad_pcb (KiCad board)
At the start: 2 copper layers, 57.9 x 95.1 mm, 20 parts, among them J1 Conn_01x02_Female, J2 Conn_01x02_Female, J3 Conn_01x02_Female, SW1 SW_DIP_x01, SW2 SW_DIP_x01, U1 OKL-T_6-W12N-C

Commit message: 基板データの更新
最後に更新してからのデータ全てです。
Other:
- board size 57.9 x 95.1 mm -> 57.9 x 45 mm
Changed lines of the file:
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@@
       (disableapertmacros false)
       (usegerberextensions false)
-      (usegerberattributes true)
-      (usegerberadvancedattributes true)
-      (creategerberjobfile true)
+      (usegerberattributes false)
+      (usegerberadvancedattributes false)
+      (creategerberjobfile false)
       (svguseinch false)
       (svgprecision 6)
@@
       (outputformat 1)
       (mirror false)
-      (drillshape 1)
+      (drillshape 0)
       (scaleselection 1)
-      (outputdirectory "")
+      (outputdirectory "gbr/")
     )
   )
@@
     (fp_line (start 4.95 -2.35) (end -2.45 -2.35) (layer "F.Fab") (width 0.1))
     (fp_line (start -2.45 3.4) (end 4.95 3.4) (layer "F.Fab") (width 0.1))
-    (pad "1" thru_hole roundrect (at 0 0 30) (size 1.7 2) (drill 1) (layers *.Cu *.Mask) (roundrect_rratio 0.147059)
+    (pad "1" thru_hole roundrect (at 0 0 30) (size 1.7 2) (drill 1) (layers *.Cu *.Mask) (roundrect_rratio 0.1470588235)
       (net 3 "+7.5V") (pinfunction "Pin_1") (pintype "passive"))
     (pad "2" thru_hole oval (at 2.5 0 30) (size 1.7 2) (drill 1) (layers *.Cu *.Mask)
@@
     (fp_line (start 4.71 -3.7) (end 4.71 -2) (layer "F.Fab") (width 0.1))
     (fp_line (start -0.75 -3.7) (end 4.71 -3.7) (layer "F.Fab") (width 0.1))
-    (pad "1" thru_hole roundrect (at 0 0 315) (size 2.7 2.7) (drill 1.7) (layers *.Cu *.Mask) (roundrect_rratio 0.092593)
+    (pad "1" thru_hole roundrect (at 0 0 315) (size 2.7 2.7) (drill 1.7) (layers *.Cu *.Mask) (roundrect_rratio 0.09259296296)
       (net 1 "Net-(BT1-Pad1)") (pinfunction "+") (pintype "passive"))
     (pad "2" thru_hole circle (at 3.96 0 315) (size 2.7 2.7) (drill 1.7) (layers *.Cu *.Mask)
@@
     (fp_line (start 4.95 -2.35) (end -2.45 -2.35) (layer "F.Fab") (width 0.1))
     (fp_line (start 4.95 3.4) (end 4.95 -2.35) (layer "F.Fab") (width 0.1))
-    (pad "1" thru_hole roundrect (at 0 0 30) (size 1.7 2) (drill 1) (layers *.Cu *.Mask) (roundrect_rratio 0.147059)
+    (pad "1" thru_hole roundrect (at 0 0 30) (size 1.7 2) (drill 1) (layers *.Cu *.Mask) (roundrect_rratio 0.1470588235)
       (net 3 "+7.5V") (pinfunction "Pin_1") (pintype "passive"))
     (pad "2" thru_hole oval (at 2.5 0 30) (size 1.7 2) (drill 1) (layers *.Cu *.Mask)
@@
     (fp_line (start -2.45 -2.35) (end -2.45 3.4) (layer "F.Fab") (width 0.1))
     (fp_line (start -2.45 3.4) (end 4.95 3.4) (layer "F.Fab") (width 0.1))
-    (pad "1" thru_hole roundrect (at 0 0 30) (size 1.7 2) (drill 1) (layers *.Cu *.Mask) (roundrect_rratio 0.147059)
+    (pad "1" thru_hole roundrect (at 0 0 30) (size 1.7 2) (drill 1) (layers *.Cu *.Mask) (roundrect_rratio 0.1470588235)
       (net 4 "+5V") (pinfunction "Pin_1") (pintype "passive"))
     (pad "2" thru_hole oval (at 2.5 0 30) (size 1.7 2) (drill 1) (layers *.Cu *.Mask)
@@
   (gr_line (start 167.315781 124.382796) (end 164.923061 120.238483) (layer "Edge.Cuts") (width 0.2))
   (gr_rect (start 126.746 113.792) (end 149.606 123.952) (layer "Edge.Cuts") (width 0.1) (fill none))
-  (gr_circle (center 155.73395 34.322476) (end 155.73395 34.422476) (layer "Edge.Cuts") (width 0.0001) (fill solid))
   (gr_circle (center 131.138075 86.849069) (end 131.138075 88.099069) (layer "Edge.Cuts") (width 0.2) (fill none))
   (gr_line (start 118.787621 100.613737) (end 124.621252 106.447368) (layer "Edge.Cuts") (width 0.2))
@@
       a11c9cbc-6b23-4372-be92-5489517fa5c9
       b03c9f8f-e091-4025-8f35-c4a6290036fe
-      e0c2897c-68a4-44aa-a2aa-fda96e7fcf19
       e8c32a67-d4ca-4735-ae4a-2b1ba274d2de
       ff7a968f-7640-4ce3-9f4f-aae4581d5fc1
