File: KiCad_Projects/main_board/_autosave-main board.kicad_pcb (KiCad board)
At the start: 2 copper layers, 110 x 110 mm, 77 parts, among them J1 Conn_01x04_Female, J2 Conn_01x04_Female, J3 Conn_01x02_Female, J4 Conn_01x05_Female, U1 Open MV open_mv, U10 Seeeduino_Xiao, U11 Seeeduino_Xiao, U12 TSSP58038, U13 TSSP58038, U14 TSSP58038, U15 TSSP58038, U2 type-c_sirial, U3 PIC18F26K20_ISS, U4 Akizuki_Logiv_Level_converter, U5 MPU6050, U6 TSSP58038, U7 TSSP58038, U8 TSSP58038, U9 TSSP58038

Commit message: 基板データの更新
最新バージョンの発注データの作成
最新バージョンの発注。
Other:
- board text added: "Munachu_Artemis"
- board text removed: "Munatyuu_Artemis"
Changed lines of the file:
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@@
     (aux_axis_origin 101.04 117.321895)
     (pcbplotparams
-      (layerselection 0x00010fc_ffffffff)
+      (layerselection 0x00010f0_ffffffff)
       (disableapertmacros false)
       (usegerberextensions false)
-      (usegerberattributes true)
-      (usegerberadvancedattributes true)
-      (creategerberjobfile true)
+      (usegerberattributes false)
+      (usegerberadvancedattributes false)
+      (creategerberjobfile false)
       (svguseinch false)
       (svgprecision 6)
@@
       (outputformat 1)
       (mirror false)
-      (drillshape 1)
+      (drillshape 0)
       (scaleselection 1)
-      (outputdirectory "")
+      (outputdirectory "新しいフォルダー/")
     )
   )
@@
     (fp_line (start -2.45 -3.4) (end 12.45 -3.4) (layer "B.Fab") (width 0.1))
     (fp_line (start -2.45 2.35) (end -2.45 -3.4) (layer "B.Fab") (width 0.1))
-    (pad "1" thru_hole roundrect (at 0 0 180) (size 1.7 1.95) (drill 0.95) (layers *.Cu *.Mask) (roundrect_rratio 0.147059)
+    (pad "1" thru_hole roundrect (at 0 0 180) (size 1.7 1.95) (drill 0.95) (layers *.Cu *.Mask) (roundrect_rratio 0.1470588235)
       (net 7 "GND") (pinfunction "Pin_1") (pintype "passive"))
     (pad "2" thru_hole oval (at 2.5 0 180) (size 1.7 1.95) (drill 0.95) (layers *.Cu *.Mask)
@@
     (fp_line (start -2.45 -3.4) (end 9.95 -3.4) (layer "B.Fab") (width 0.1))
     (fp_line (start 9.95 -3.4) (end 9.95 2.35) (layer "B.Fab") (width 0.1))
-    (pad "1" thru_hole roundrect (at 0 0 180) (size 1.7 1.95) (drill 0.95) (layers *.Cu *.Mask) (roundrect_rratio 0.147059)
+    (pad "1" thru_hole roundrect (at 0 0 180) (size 1.7 1.95) (drill 0.95) (layers *.Cu *.Mask) (roundrect_rratio 0.1470588235)
       (net 7 "GND") (pinfunction "Pin_1") (pintype "passive"))
     (pad "2" thru_hole oval (at 2.5 0 180) (size 1.7 1.95) (drill 0.95) (layers *.Cu *.Mask)
@@
     (fp_line (start 4.95 2.35) (end -2.45 2.35) (layer "B.Fab") (width 0.1))
     (fp_line (start -0.625 2.35) (end 0 1.35) (layer "B.Fab") (width 0.1))
-    (pad "1" thru_hole roundrect (at 0 0 90) (size 1.7 2) (drill 1) (layers *.Cu *.Mask) (roundrect_rratio 0.147059)
+    (pad "1" thru_hole roundrect (at 0 0 90) (size 1.7 2) (drill 1) (layers *.Cu *.Mask) (roundrect_rratio 0.1470588235)
       (net 7 "GND") (pinfunction "Pin_1") (pintype "passive"))
     (pad "2" thru_hole oval (at 2.5 0 90) (size 1.7 2) (drill 1) (layers *.Cu *.Mask)
@@
     (fp_line (start -2.45 2.35) (end -2.45 -3.4) (layer "B.Fab") (width 0.1))
     (fp_line (start 0 1.35) (end 0.625 2.35) (layer "B.Fab") (width 0.1))
-    (pad "1" thru_hole roundrect (at 0 0 90) (size 1.7 1.95) (drill 0.95) (layers *.Cu *.Mask) (roundrect_rratio 0.147059)
+    (pad "1" thru_hole roundrect (at 0 0 90) (size 1.7 1.95) (drill 0.95) (layers *.Cu *.Mask) (roundrect_rratio 0.1470588235)
       (net 15 "Net-(J2-Pad1)") (pinfunction "Pin_1") (pintype "passive"))
     (pad "2" thru_hole oval (at 2.5 0 90) (size 1.7 1.95) (drill 0.95) (layers *.Cu *.Mask)
@@
     (effects (font (size 1 1) (thickness 0.15)))
   )
-  (gr_text "Munatyuu_Artemis" (at 101.346 68.326 180) (layer "F.SilkS")
+  (gr_text "Munachu_Artemis" (at 101.346 68.326 180) (layer "F.SilkS")
     (effects (font (size 1.5 1.5) (thickness 0.3)))
   )
-  (gr_text "Munatyuu_Artemis" (at 101.6 166.116) (layer "F.SilkS")
+  (gr_text "Munachu_Artemis" (at 101.6 166.116) (layer "F.SilkS")
     (effects (font (size 1.5 1.5) (thickness 0.3)))
   )
