File: KiCad_Projects/2022 late/Teensy_ver/IO_Board_Teensy/IO_Board.kicad_pcb (KiCad board)
At the start: 2 copper layers, 85.4 x 99.1 mm, 40 parts, among them J1 USB_C_Receptacle_USB2.0, J10 USB_C_Receptacle_USB2.0, J2 Conn_01x06_Female, J3 Conn_01x10_Female, J4 USB_C_Receptacle_USB2.0, J5 Conn_01x10_Female, J6 Conn_01x17_Female, J7 USB_C_Receptacle_USB2.0, J8 Conn_01x10_Female, J9 Conn_01x06_Female

Commit message: 基板データの更新
1318のファイルがたまってました
多くなって申し訳ない
Parts:
- moved J5 3.81 mm to (163.8, 81.0)
- moved J8 3.81 mm to (163.8, 77.2)
Routing:
- net Line D+: track 69.1 -> 2.93 mm
- net Line D-: track 68.0 -> 2.69 mm
- net +3V3: track 158.7 -> 96.2 mm, vias 6 -> 3
- net +5V: track 163.1 -> 100.7 mm
- net stop: track 78.1 -> 16.7 mm, vias 1 -> 0
- net Reset 1: track 58.7 -> 0.00 mm
- net Teensy D+: track 75.7 -> 17.8 mm
- net MOSI 2: track 57.7 -> 0.00 mm
- net Teensy D-: track 73.9 -> 16.7 mm
- net Cam D+: track 89.4 -> 32.9 mm
- net SCK 2: track 59.3 -> 3.59 mm
- net Cam D-: track 88.5 -> 32.7 mm
- net MISO 1: track 58.0 -> 6.20 mm
- net MOSI 1: track 51.6 -> 2.69 mm
- net SCK 1: track 50.8 -> 3.32 mm
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- removed copper zone on B.Cu, net GND
- removed copper zone on F.Cu, net GND
